File: hardware/radar60.kicad_pcb (KiCad board)
At the start: 2 copper layers, 0 parts

Commit message: PCB: sincronizada con el esquema, contorno circular de 60 mm y colocación de la cara superior
Parts:
- added C1: 4.7u, Capacitor_SMD:C_0805_2012Metric, F.Cu at (84.3, 106.0)
- added C10: 100n, Capacitor_SMD:C_0402_1005Metric, F.Cu at (5.91, 57.4)
- added C11: 100n, Capacitor_SMD:C_0402_1005Metric, F.Cu at (5.91, 63.4)
- added C12: 1u, Capacitor_SMD:C_0402_1005Metric, F.Cu at (5.91, 69.4)
- added C13: 100n, Capacitor_SMD:C_0402_1005Metric, F.Cu at (5.91, 75.4)
- added C14: 1u, Capacitor_SMD:C_0402_1005Metric, F.Cu at (5.91, 81.4)
- added C15: 100n, Capacitor_SMD:C_0402_1005Metric, F.Cu at (5.91, 87.4)
- added C16: 100n, Capacitor_SMD:C_0402_1005Metric, F.Cu at (5.91, 93.4)
- added C17: 100n, Capacitor_SMD:C_0402_1005Metric, F.Cu at (5.91, 99.4)
- added C18: 100n, Capacitor_SMD:C_0402_1005Metric, F.Cu at (99.8, 91.0)
- added C19: 100n, Capacitor_SMD:C_0402_1005Metric, F.Cu at (108.2, 91.0)
- added C2: 10u, Capacitor_SMD:C_0805_2012Metric, F.Cu at (91.7, 106.0)
- added C20: 100n, Capacitor_SMD:C_0402_1005Metric, F.Cu at (99.8, 99.5)
- added C21: 100n, Capacitor_SMD:C_0402_1005Metric, F.Cu at (108.2, 99.5)
- added C22: 10u, Capacitor_SMD:C_0805_2012Metric, F.Cu at (6.70, 129.9)
- added C23: 100n, Capacitor_SMD:C_0402_1005Metric, F.Cu at (5.91, 136.3)
- added C24: 100n, Capacitor_SMD:C_0402_1005Metric, F.Cu at (119.8, 104.0)
- added C25: 1u, Capacitor_SMD:C_0402_1005Metric, F.Cu at (121.3, 104.0)
- added C26: 100n, Capacitor_SMD:C_0402_1005Metric, F.Cu at (115.5, 109.5)
- added C3: 1u, Capacitor_SMD:C_0402_1005Metric, F.Cu at (84.8, 97.0)
- added C4: 10u, Capacitor_SMD:C_0805_2012Metric, F.Cu at (91.7, 97.0)
- added C5: 100n, Capacitor_SMD:C_0402_1005Metric, F.Cu at (5.91, 27.4)
- added C6: 100n, Capacitor_SMD:C_0402_1005Metric, F.Cu at (5.91, 33.4)
- added C7: 100n, Capacitor_SMD:C_0402_1005Metric, F.Cu at (5.91, 39.4)
- added C8: 1u, Capacitor_SMD:C_0402_1005Metric, F.Cu at (5.91, 45.4)
- added C9: 100n, Capacitor_SMD:C_0402_1005Metric, F.Cu at (5.91, 51.4)
- added D1: LED_RGB_CA, LED_SMD:LED_RGB_1210, F.Cu at (7.90, 162.1)
- added F1: 500mA, Fuse:Fuse_1206_3216Metric, F.Cu at (108.0, 115.5)
- added FB1: 600R@100MHz, Inductor_SMD:L_0603_1608Metric, F.Cu at (6.48, 177.3)
- added FB2: 600R@100MHz, Inductor_SMD:L_0603_1608Metric, F.Cu at (6.48, 183.7)
- added FB3: 600R@100MHz, Inductor_SMD:L_0603_1608Metric, F.Cu at (6.48, 190.2)
- added FB4: 600R@100MHz, Inductor_SMD:L_0603_1608Metric, F.Cu at (84.5, 101.5)
- added J1: GT-USB-7051A, Connector_USB:USB_C_Receptacle_G-Switch_GT-USB-7051x, F.Cu at (100.0, 116.0)
- added J2: Conn_ARM_SWD_TagConnect_TC2030-NL, Connector:Tag-Connect_TC2030-IDC-NL_2x03_P1.27mm_Vertical, F.Cu at (80.0, 113.0)
- added R1: 5.1k, Resistor_SMD:R_0402_1005Metric, F.Cu at (95.5, 121.0)
- added R10: 1k, Resistor_SMD:R_0402_1005Metric, F.Cu at (97.5, 126.0)
- added R11: 1k, Resistor_SMD:R_0402_1005Metric, F.Cu at (100.0, 127.0)
- added R12: 1k, Resistor_SMD:R_0402_1005Metric, F.Cu at (102.5, 126.0)
- added R2: 5.1k, Resistor_SMD:R_0402_1005Metric, F.Cu at (104.5, 121.0)
- added R3: 100k, Resistor_SMD:R_0402_1005Metric, F.Cu at (88.0, 93.6)
- added R4: 22, Resistor_SMD:R_0402_1005Metric, F.Cu at (5.93, 241.3)
- added R5: 10k, Resistor_SMD:R_0402_1005Metric, F.Cu at (5.93, 247.3)
- added R6: 10k, Resistor_SMD:R_0402_1005Metric, F.Cu at (5.93, 253.3)
- added R7: 22.1k, Resistor_SMD:R_0402_1005Metric, F.Cu at (120.5, 98.5)
- added R8: 47.5k, Resistor_SMD:R_0402_1005Metric, F.Cu at (122.0, 98.5)
- added R9: 1k, Resistor_SMD:R_0402_1005Metric, F.Cu at (115.5, 100.0)
- added SW1: PUESTA_EN_MARCHA, Button_Switch_SMD:SW_SPST_TL3342, F.Cu at (82.5, 87.5)
- added SW2: RESET, Button_Switch_SMD:SW_SPST_TL3342, F.Cu at (117.5, 87.5)
- added TP1: TP, TestPoint:TestPoint_Pad_D1.0mm, F.Cu at (111.5, 120.5)
- added TP10: TP, TestPoint:TestPoint_Pad_D1.0mm, F.Cu at (89.5, 83.5)
- added TP11: TP, TestPoint:TestPoint_Pad_D1.0mm, F.Cu at (90.0, 86.5)
- added TP12: TP, TestPoint:TestPoint_Pad_D1.0mm, F.Cu at (90.0, 89.0)
- added TP2: TP, TestPoint:TestPoint_Pad_D1.0mm, F.Cu at (79.5, 105.0)
- added TP3: TP, TestPoint:TestPoint_Pad_D1.0mm, F.Cu at (79.5, 97.0)
- added TP4: TP, TestPoint:TestPoint_Pad_D1.0mm, F.Cu at (124.5, 109.0)
- added TP5: TP, TestPoint:TestPoint_Pad_D1.0mm, F.Cu at (110.5, 89.5)
- added TP6: TP, TestPoint:TestPoint_Pad_D1.0mm, F.Cu at (112.5, 91.0)
- added TP7: TP, TestPoint:TestPoint_Pad_D1.0mm, F.Cu at (110.5, 97.5)
- added TP8: TP, TestPoint:TestPoint_Pad_D1.0mm, F.Cu at (112.5, 94.0)
- added TP9: TP, TestPoint:TestPoint_Pad_D1.0mm, F.Cu at (110.5, 103.0)
- added U1: BGT60TR13C, radar60:Infineon_PG-VF2BGA-40-1_6.5x5mm_P0.5mm, F.Cu at (8.88, 417.8)
- added U2: MGM260PB32VNA, radar60:SiliconLabs_MGM260P_12.9x15mm, F.Cu at (100.0, 78.5)
- added U3: AP2112K-3.3, Package_TO_SOT_SMD:SOT-23-5, F.Cu at (88.0, 106.0)
- added U4: AP2112K-1.8, Package_TO_SOT_SMD:SOT-23-5, F.Cu at (88.0, 97.0)
- added U5: CP2102N-A02-GQFN24, Package_DFN_QFN:QFN-24-1EP_4x4mm_P0.5mm_EP2.6x2.6mm, F.Cu at (115.5, 105.0)
- added U6: USBLC6-2SC6, Package_TO_SOT_SMD:SOT-23-6, F.Cu at (93.0, 115.5)
- added U7: SN74AVC4T245PW, Package_SO:TSSOP-16_4.4x5mm_P0.65mm, F.Cu at (104.0, 93.0)
- added U8: SN74AVC4T245PW, Package_SO:TSSOP-16_4.4x5mm_P0.65mm, F.Cu at (104.0, 101.5)
- added Y1: SiT8008BI-12-18E-80.000000, Oscillator:Oscillator_SMD_SiT_PQFN-4Pin_2.5x2.0mm, F.Cu at (6.76, 505.2)
Other:
- board outline added: 60 x 60 mm
