File: hardware/radar60.kicad_pcb (KiCad board)
At the start: 2 copper layers, 60 x 60 mm, 69 parts, among them J1 GT-USB-7051A, J2 Conn_ARM_SWD_TagConnect_TC203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, SW1 PUESTA_EN_MARCHA, SW2 RESET, U1 BGT60TR13C, U2 MGM260PB32VNA, U3 AP2112K-3.3, U4 AP2112K-1.8, U5 CP2102N-A02-GQFN24, U6 USBLC6-2SC6, U7 SN74AVC4T245PW, U8 SN74AVC4T245PW, Y1 SiT8008BI-12-18E-80.000000

Commit message: PCB rev A terminada: 4 capas, rutada, DRC limpia y ficheros de fabricación
- Apilado JLC04161H-7628: F.Cu señal, In1 GND entero, In2 alimentación con
  relleno de GND, B.Cu radar; zonas prohibidas de la antena del MGM260P, de In2
  bajo el radar y de los apoyos de la carcasa
- Cara inferior: BGT60TR13C centrado en el radomo, desacoplos directos a cada
  bola, ferritas y bulk por raíl, reloj de 80 MHz de 6,3 mm en B.Cu
- Fan-out del BGA sin vía en pad; resto con Freerouting (GND por planos) y
  ~490 vías de cosido validadas con la DRC
- Huellas refrescadas desde biblioteca (atributo SMD, modelos 3D; tetones de
  J1 respetados); envolventes 3D propias para radar, módulo, USB-C y oscilador
- Esquema: puntos de prueba y Tag-Connect fuera de la BOM
- ERC 0, DRC 0 errores, 0 sin conectar, 0 diferencias con el esquema
- scripts/fabricacion.sh: Gerber, taladros, BOM/CPL JLCPCB, PDF y STEP

Co-Authored-By: Claude Opus 5.5 <noreply@anthropic.com>
Claude-Session: https://claude.ai/code/session_01G1CWE6SnEXSgcHy8fSbaPj
Parts:
- C10, C11, C12, C13, C14, C15, C16, C17, C5, C6, C7, C8, C9, D1, FB1, FB2, FB3, R4, U1, Y1: moved to B.Cu
- moved Y1 409.3 mm to (105.6, 108.0), turned to 180 degrees
- moved U1 330.6 mm to (100.0, 100.0), turned to -90 degrees
- moved R6 189.1 mm to (109.6, 95.1), turned to 180 degrees
- moved R5 185.1 mm to (109.6, 94.0), turned to 180 degrees
- moved R4 166.0 mm to (102.0, 105.9), turned to 90 degrees
- moved FB3 136.4 mm to (107.6, 98.6), turned to -90 degrees
- moved FB2 130.0 mm to (107.6, 102.0), turned to 90 degrees
- moved C5 124.9 mm to (103.0, 105.9), turned to -90 degrees
- moved C6 118.8 mm to (100.0, 105.9), turned to -90 degrees
- moved FB1 114.5 mm to (95.3, 105.0)
- moved C7 114.4 mm to (99.0, 105.9), turned to -90 degrees
- moved C12 108.0 mm to (108.9, 102.0), turned to -90 degrees
- moved C11 106.6 mm to (105.4, 101.6)
- moved C8 106.5 mm to (95.7, 102.6), turned to 180 degrees
- moved C23 105.1 mm to (99.1, 87.7)
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Routing:
- net /+3V3: track 0.00 -> 140.2 mm, vias 0 -> 1
- net /NRST: track 0.00 -> 84.4 mm, vias 0 -> 2
- net /LED_B: track 0.00 -> 59.0 mm, vias 0 -> 2
- net /LED_G: track 0.00 -> 57.0 mm, vias 0 -> 2
- net /GND: track 0.00 -> 55.5 mm, vias 0 -> 425
- net /LED_R: track 0.00 -> 54.7 mm, vias 0 -> 2
- net /VBUS: track 0.00 -> 53.0 mm, vias 0 -> 2
- net /VCOM_RX: track 0.00 -> 47.7 mm, vias 0 -> 2
- net /+1V8_D: track 0.00 -> 47.5 mm, vias 0 -> 2
- net /+1V8_RAD: track 0.00 -> 47.1 mm, vias 0 -> 2
- net /VCOM_TX: track 0.00 -> 46.3 mm, vias 0 -> 2
- net /USB_DP: track 0.00 -> 43.2 mm, vias 0 -> 2
- net /SWDIO: track 0.00 -> 43.1 mm, vias 0 -> 2
- net /SWCLK: track 0.00 -> 42.0 mm, vias 0 -> 2
- net /SWO: track 0.00 -> 38.5 mm, vias 0 -> 2
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- added copper zone on B.Cu, net /GND
- added copper zone on F.Cu, net /GND
- added copper zone on In1.Cu, net /GND
- added copper zone on In2.Cu, net /GND
Other:
- copper layers 2 -> 4

Commit message: Hardware: revisión con las hojas de datos de los fabricantes
- Radar (hoja BGT60TR13C y placa de referencia de Infineon): VAREF 470 nF,
  desacoplos por dominio como la referencia, LDO de 1,8 V de bajo ruido
  (TPS7A2018, mismo patillaje), VDDLF con filtro RC (R13 47 ohm + 10 uF),
  serie del reloj 150 ohm y pads del BGA a 0,275 mm
- Reloj: el SiT8008 (MEMS) no cumple el jitter de 1 ps; pasa a cuarzo Kyocera
  KC2520K con el mismo patrón 2520
- MGM260P: código completo MGM260PB22VNA5 (+10 dBm); patillaje, patrón y
  zona de antena verificados; altura 2,35 mm
- USB-C a 7,5 mm de altura; CP2102N con 4,7 uF
- ERC 0, DRC 0, sin diferencias esquema-placa; mecánica sin interferencias
- docs/09: tabla de verificación, BOM rev A, balance y riesgos para F2

Co-Authored-By: Claude Opus 5.5 <noreply@anthropic.com>
Claude-Session: https://claude.ai/code/session_01G1CWE6SnEXSgcHy8fSbaPj
Parts:
- removed FB4: 600R@100MHz, Inductor_SMD:L_0603_1608Metric
- added R13: 47, Resistor_SMD:R_0603_1608Metric, F.Cu at (84.5, 101.5)
- C10, C17, C9: value 100n -> 1u
- C12, C8: value 1u -> 10u
- C15: value 100n -> 10u
- C16: value 100n -> 470n
- C25: value 1u -> 4.7u
- R4: value 22 -> 150
- U2: value MGM260PB32VNA -> MGM260PB22VNA5
- U4: value AP2112K-1.8 -> TPS7A2018PDBVR
- Y1: value SiT8008BI-12-18E-80.000000 -> KC2520K80.0000
