File: hardware/radar60.kicad_sch (KiCad schematic)
At the start: 69 parts, among them J1 GT-USB-7051A, J2 Conn_ARM_SWD_TagConnect_TC203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, SW1 PUESTA_EN_MARCHA, SW2 RESET, U1 BGT60TR13C, U2 MGM260PB32VNA, U3 AP2112K-3.3, U4 AP2112K-1.8, U5 CP2102N-A02-GQFN24, U6 USBLC6-2SC6, U7 SN74AVC4T245PW, U8 SN74AVC4T245PW, Y1 SiT8008BI-12-18E-80.000000

Commit message: PCB rev A terminada: 4 capas, rutada, DRC limpia y ficheros de fabricación
- Apilado JLC04161H-7628: F.Cu señal, In1 GND entero, In2 alimentación con
  relleno de GND, B.Cu radar; zonas prohibidas de la antena del MGM260P, de In2
  bajo el radar y de los apoyos de la carcasa
- Cara inferior: BGT60TR13C centrado en el radomo, desacoplos directos a cada
  bola, ferritas y bulk por raíl, reloj de 80 MHz de 6,3 mm en B.Cu
- Fan-out del BGA sin vía en pad; resto con Freerouting (GND por planos) y
  ~490 vías de cosido validadas con la DRC
- Huellas refrescadas desde biblioteca (atributo SMD, modelos 3D; tetones de
  J1 respetados); envolventes 3D propias para radar, módulo, USB-C y oscilador
- Esquema: puntos de prueba y Tag-Connect fuera de la BOM
- ERC 0, DRC 0 errores, 0 sin conectar, 0 diferencias con el esquema
- scripts/fabricacion.sh: Gerber, taladros, BOM/CPL JLCPCB, PDF y STEP

Co-Authored-By: Claude Opus 5.5 <noreply@anthropic.com>
Claude-Session: https://claude.ai/code/session_01G1CWE6SnEXSgcHy8fSbaPj
Parts:
- J2, TP1, TP10, TP11, TP12, TP2, TP3, TP4, TP5, TP6, TP7, TP8, TP9: now left out of the parts list
Changed lines of the file:
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@@
 		(at 398.78 160.02 0)
 		(unit 1)
-		(in_bom yes)
+		(in_bom no)
 		(on_board yes)
 		(dnp no)
@@
 		(at 482.6 83.82 0)
 		(unit 1)
-		(in_bom yes)
+		(in_bom no)
 		(on_board yes)
 		(dnp no)
@@
 		(at 502.92 83.82 0)
 		(unit 1)
-		(in_bom yes)
+		(in_bom no)
 		(on_board yes)
 		(dnp no)
@@
 		(at 482.6 96.52 0)
 		(unit 1)
-		(in_bom yes)
+		(in_bom no)
 		(on_board yes)
 		(dnp no)
@@
 		(at 502.92 96.52 0)
 		(unit 1)
-		(in_bom yes)
+		(in_bom no)
 		(on_board yes)
 		(dnp no)
@@
 		(at 482.6 109.22 0)
 		(unit 1)
-		(in_bom yes)
+		(in_bom no)
 		(on_board yes)
 		(dnp no)
@@
 		(at 502.92 109.22 0)
 		(unit 1)
-		(in_bom yes)
+		(in_bom no)
 		(on_board yes)
 		(dnp no)
@@
 		(at 482.6 121.92 0)
 		(unit 1)
-		(in_bom yes)
+		(in_bom no)
 		(on_board yes)
 		(dnp no)
@@
 		(at 502.92 121.92 0)
 		(unit 1)
-		(in_bom yes)
+		(in_bom no)
 		(on_board yes)
 		(dnp no)
@@
 		(at 482.6 134.62 0)
 		(unit 1)
-		(in_bom yes)
+		(in_bom no)
 		(on_board yes)
 		(dnp no)
@@
 		(at 502.92 134.62 0)
 		(unit 1)
-		(in_bom yes)
+		(in_bom no)
 		(on_board yes)
 		(dnp no)
@@
 		(at 482.6 147.32 0)
 		(unit 1)
-		(in_bom yes)
+		(in_bom no)
 		(on_board yes)
 		(dnp no)
@@
 		(at 502.92 147.32 0)
 		(unit 1)
-		(in_bom yes)
-		(on_board yes)
-		(dnp no)
+		(in_bom no)
+		(on_board yes)
+		(dnp no)

Commit message: Hardware: revisión con las hojas de datos de los fabricantes
- Radar (hoja BGT60TR13C y placa de referencia de Infineon): VAREF 470 nF,
  desacoplos por dominio como la referencia, LDO de 1,8 V de bajo ruido
  (TPS7A2018, mismo patillaje), VDDLF con filtro RC (R13 47 ohm + 10 uF),
  serie del reloj 150 ohm y pads del BGA a 0,275 mm
- Reloj: el SiT8008 (MEMS) no cumple el jitter de 1 ps; pasa a cuarzo Kyocera
  KC2520K con el mismo patrón 2520
- MGM260P: código completo MGM260PB22VNA5 (+10 dBm); patillaje, patrón y
  zona de antena verificados; altura 2,35 mm
- USB-C a 7,5 mm de altura; CP2102N con 4,7 uF
- ERC 0, DRC 0, sin diferencias esquema-placa; mecánica sin interferencias
- docs/09: tabla de verificación, BOM rev A, balance y riesgos para F2

Co-Authored-By: Claude Opus 5.5 <noreply@anthropic.com>
Claude-Session: https://claude.ai/code/session_01G1CWE6SnEXSgcHy8fSbaPj
Parts:
- C10, C17, C9: value 100n -> 1u
- C12, C8: value 1u -> 10u
- C15: value 100n -> 10u
- C16: value 100n -> 470n
- C25: value 1u -> 4.7u
- R13: renamed from FB4; value 600R@100MHz -> 47; footprint Inductor_SMD:L_0603_1608Metric -> Resistor_SMD:R_0603_1608Metric; symbol Device:FerriteBead_Small -> Device:R_Small
- R4: value 22 -> 150
- U2: value MGM260PB32VNA -> MGM260PB22VNA5
- U4: value AP2112K-1.8 -> TPS7A2018PDBVR
- Y1: value SiT8008BI-12-18E-80.000000 -> KC2520K80.0000
Changed lines of the file:
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@@
 			)
 		)
-		(property "Value" "AP2112K-1.8"
+		(property "Value" "TPS7A2018PDBVR"
 			(at 187.96 42.545 0)
 			(effects
@@
 			)
 		)
-		(property "Datasheet" "https://www.diodes.com/assets/Datasheets/AP2112.pdf"
+		(property "Datasheet" "https://www.ti.com/lit/ds/symlink/tps7a20.pdf"
 			(at 187.96 48.26 0)
 			(hide yes)
@@
 	)
 	(symbol
-		(lib_id "Device:FerriteBead_Small")
+		(lib_id "Device:R_Small")
 		(at 228.6 71.12 90)
 		(unit 1)
@@
 		(on_board yes)
 		(dnp no)
-		(property "Reference" "FB4"
+		(property "Reference" "R13"
 			(at 227.33 69.215 0)
 			(effects
@@
 			)
 		)
-		(property "Value" "600R@100MHz"
+		(property "Value" "47"
 			(at 229.87 69.215 0)
 			(effects
@@
 			)
 		)
-		(property "Footprint" "Inductor_SMD:L_0603_1608Metric"
+		(property "Footprint" "Resistor_SMD:R_0603_1608Metric"
 			(at 228.6 71.12 0)
 			(hide yes)
@@
 			)
 		)
-		(property "Description" "Ferrite bead, small symbol"
+		(property "Description" "Resistor, small symbol"
 			(at 228.6 71.12 0)
 			(hide yes)
@@
 			(project "radar60"
 				(path "/544589c5-c7ce-44b5-b5ae-1d336c726c76"
-					(reference "FB4")
+					(reference "R13")
 					(unit 1)
 				)
@@
 			)
 		)
-		(property "Value" "SiT8008BI-12-18E-80.000000"
+		(property "Value" "KC2520K80.0000"
 			(at 261.366 150.622 0)
 			(effects
@@
 			)
 		)
-		(property "Datasheet" "https://www.sitime.com/support/resource-library/datasheets/sit8008-datasheet"
+		(property "Datasheet" ""
 			(at 248.92 157.48 0)
 			(hide yes)
@@
 			)
 		)
-		(property "Value" "22"
+		(property "Value" "150"
 			(at 271.78 157.48 90)
 			(effects
@@
 			)
 		)
-		(property "Value" "100n"
+		(property "Value" "1u"
 			(at 236.855 160.02 0)
 			(effects
@@
 			)
 		)
-		(property "Value" "MGM260PB32VNA"
+		(property "Value" "MGM260PB22VNA5"
 			(at 101.6 210.82 0)
 			(effects
@@
 			)
 		)
-		(property "Value" "1u"
+		(property "Value" "4.7u"
 			(at 432.435 45.72 0)
 			(effects
@@
 			)
 		)
-		(property "Value" "1u"
+		(property "Value" "10u"
 			(at 277.495 281.94 0)
 			(effects
@@
 			)
 		)
-		(property "Value" "100n"
+		(property "Value" "1u"
 			(at 285.115 281.94 0)
 			(effects
@@
 			)
 		)
-		(property "Value" "100n"
+		(property "Value" "1u"
 			(at 292.735 281.94 0)
 			(effects
@@
 			)
 		)
-		(property "Value" "1u"
+		(property "Value" "10u"
 			(at 307.975 281.94 0)
 			(effects
@@
 			)
 		)
-		(property "Value" "100n"
+		(property "Value" "10u"
 			(at 330.835 281.94 0)
 			(effects
@@
 			)
 		)
-		(property "Value" "100n"
+		(property "Value" "470n"
 			(at 338.455 281.94 0)
 			(effects
